File: FC_Board/FC.kicad_sch (KiCad schematic)
At the start: 77 parts, among them J1 Programmer_pins, J2 Pyro1, J3 Pyro2, J4 Pyro3, J5 Pyro4, J6 Conn_01x03, J7 Conn_01x03, J8 MEM2090-00-145-00-A_REVA, M1 Motor_Servo, M2 Motor_Servo, M3 Motor_Servo, M4 Motor_Servo, Q1 PMOS, Q2 NMOS, Q3 NMOS, Q4 NMOS, Q5 NMOS, U1 PIC32MZ2048EFH100-I/PF, U2 LM7805MPX/NOPB, U3 LDL1117S33R, U4 LSM6DS3TR-C, U5 LIS3MDLTR, U6 MS5607-02BA, U7 NEO-M8Q, U8 SST26VF032BT-104I/SM, U9 INA219AxD

Commit message: Schematic update
- Add: PWM level shifting
- Add: SPI bus
- Add: buzzer drain setup
- Update: 5V power for servos
- Verify: LDO sizing
Parts:
- added U10, U11, U12, U13: SN74AHCT1G125DCKR, SN74AHCT1G125DCKR:SOT65P210X110-5N, symbol SN74AHCT1G125DCKR:SN74AHCT1G125DCKR
- F1: value Fuse -> 1.5 A
- R7: value R -> 300
Connections:
- net SERVO_+ is gone; now on net 5V: M1.2 (+), M2.2 (+), M3.2 (+), M4.2 (+)
- net 3V3: now also BZ1.1 (+), D2.2 (A)
- net 5V: now also U10.5 (VCC), U11.5 (VCC), U12.5 (VCC), U13.5 (VCC)
- net Buzzer_pin: now also BZ1.2 (-), R7.1, U1.77 (EBID14/ETXEN/RPD2/PMD14/RD2); no longer BZ1.1 (+), D2.2 (A)
- net GND: now also U10.1 (~{OE}), U10.3 (GND), U11.1 (~{OE}), U11.3 (GND), U12.1 (~{OE}), U12.3 (GND), U13.1 (~{OE}), U13.3 (GND); no longer BZ1.2 (-), R7.1
- net SERVO_1: now also U10.2 (A); no longer M1.1 (PWM)
- net SERVO_2: now also U11.2 (A); no longer M2.1 (PWM)
- net SERVO_3: now also U12.2 (A); no longer M3.1 (PWM)
- net SERVO_4: now also U13.2 (A); no longer M4.1 (PWM)
- new net: M1.1 (PWM), U10.4 (Y)
- new net: M2.1 (PWM), U11.4 (Y)
- new net: M3.1 (PWM), U12.4 (Y)
- new net: M4.1 (PWM), U13.4 (Y)
Other:
- note added: "(com level shifting)"
- note added: "Notas: - Conectores para ler flash memory - Interrupts. NC ou GND? - Pull-ups (I2C altímetro. Colocar como opcional, shunts) - Sou capaz de precisar de mais reguladores de tensão para ter corrente suficiente - Ligar flash memory ao GPS - Antena activa ou passiva (GPS)? - Verificar valores de decouplers - O MCU escolhido está bastante overpowered para a aplicação - Não esquecer SPI altímetro e GPS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"
- note added: "OVERALL"
- note added: "SPI CLK"
- note added: "SPI MISO"
- note added: "SPI MOSI"
- note added: "SPI separado também. Partilhado apenas com logging"
- note added: "open drain"
- note removed: "Convém confirmar se PIC consegue dar drive do buzzer e led simultaneamente, talvez fosse boa ideia usar open drain type config"
- note removed: "Ligar a GPIO's"
- note removed: "MCU - 3V3 GPS - 3V3 IMU - 1.8V? (3.6max) Magnetómetro - 3V3 Altímetro - 3V3"
- note removed: "Notas: - 5V necessário? - Calcular Pull resistors do SPI - Conectores para ler flash memory - Adicionar possibilidade de ter resistências série para linhas de transmissão - Interrupts? - Pull-ups nos clocks? (I2C) - Sou capaz de precisar de mais reguladores de tensão para ter corrente suficiente - Ligar flash memory ao GPS - Antena activa ou passiva (GPS)? - Verificar valores de decouplers"
- note removed: "Provavelmente vou ter de mudar isto para um com Vdrop menor. Só preciso de 5V talvez para a antena anyways"

Commit message: Schematic update
- Remove: Buffers on PWM unnecessary (internal servo logic handles 3V3)
- Add: Selecting PIC pins for SPI bus and sensor interrupts
- Other minor tweaks
Parts:
- removed U10, U11, U12, U13: SN74AHCT1G125DCKR, SN74AHCT1G125DCKR:SOT65P210X110-5N, symbol SN74AHCT1G125DCKR:SN74AHCT1G125DCKR
- added Q6: NMOS, symbol Simulation_SPICE:NMOS
- added R13, R14, R15, R16, R17: 10k, symbol Device:R
- D1: value -10V -> 10V
- R7: value 300 -> 150
Connections:
- net Buzzer_pin: now also Q6.2 (G), R17.2; no longer BZ1.2 (-), R7.1
- net GND: now also Q6.3 (S), R13.1, R14.1, R15.1, R16.1, R17.1
- net Pyro_channel1: now also R14.2
- net Pyro_channel2: now also R13.2
- net Pyro_channel3: now also R15.2
- net Pyro_channel4: now also R16.2
- net SERVO_1: now also M1.1 (PWM)
- net SERVO_2: now also M2.1 (PWM)
- net SERVO_3: now also M3.1 (PWM)
- net SERVO_4: now also M4.1 (PWM)
- net SPI_CLK: now also U1.76 (RPD1/SCK1/RD1)
- net SPI_MISO: now also U1.73 (SOSCO/RPC14/T1CK/RC14)
- net SPI_MOSI: now also U1.72 (SOSCI/RPC13/RC13)
- net IMU_INT1: now reaches U4.4 (INT1)
- net IMU_INT1: now also U1.100 (EBID4/AN18/PMD4/RE4)
- net IMU_INT2: now reaches U4.9 (INT2)
- net IMU_INT2: now also U1.99 (EBID3/RPE3/PMD3/RE3)
- net MAG_DR: now reaches U1.96 (TRD1/SQID1/RG12)
- net MAG_DR: now also U5.8 (DRDY)
- net MAG_INT: now reaches U1.97 (TRD0/SQID0/RG13)
- net MAG_INT: now also U5.7 (INT)
- new net: BZ1.2 (-), Q6.1 (D), R7.1
Other:
- note added: "Aqui tenho de usar switching mosfets bons"
- note added: "Minimizar RdsON"
- note added: "Notas: - Conectores para ler flash memory - Pull-ups (I2C altímetro. Colocar como opcional, shunts) - Ligar flash memory ao GPS - Antena activa ou passiva (GPS)? - Verificar valores de decouplers - O MCU escolhido está bastante overpowered para a aplicação - Não esquecer SPI altímetro e GPS(são separados)"
- note added: "Zener dá clamp para cumprir máx vgs quando reverse polarity"
- note removed: "(com level shifting)"
- note removed: "Notas: - Conectores para ler flash memory - Interrupts. NC ou GND? - Pull-ups (I2C altímetro. Colocar como opcional, shunts) - Sou capaz de precisar de mais reguladores de tensão para ter corrente suficiente - Ligar flash memory ao GPS - Antena activa ou passiva (GPS)? - Verificar valores de decouplers - O MCU escolhido está bastante overpowered para a aplicação - Não esquecer SPI altímetro e GPS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"
- note removed: "OVERALL"
- note removed: "REVERSE POLARITY PROTECTION Substituir por schottky?"
- note removed: "Tenho de decidir qual das linhas quero monitorizar. Overall power?PIC?... Suponho que nada me impede ter vários ICs a ver linhas diferentes mas parece-me excessivo."
- note removed: "Transistores chegam a abrir completamente se a tensão da bateria fôr superior à tensão aplicada pelo PIC na gate?"
- note removed: "open drain"
- moved on the sheet: BZ1, C14, C16, C22, C23, C24, C25, C26, C5, C7, D2, J2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

Commit message: Power monitoring done
Parts:
- removed C31: C, symbol Device:C
- removed R10, R9: R, symbol Device:R
- added R18, R19, R20, R21: 10k, symbol Device:R
- R8: value R_Shunt -> 0.04
Connections:
- net 3V3: now also R18.2, R19.2, R20.2, R21.2
- net FLASH_EN: now also R21.1
- net GND: now also U9.1 (A1), U9.2 (A0)
- net GPS_CS: now also R20.1
- net PWR_SDA: now also U1.5 (EBID7/AN15/PMD7/RE7), R18.1
- net PWR_SDL: now also U1.4 (EBID6/AN16/PMD6/RE6), R19.1
- net Shunt_OUT: now reaches C18.1, C20.1, U2.1 (VI), U3.3 (VIN)
- net Shunt_OUT: now also R8.1; no longer D1.1 (K), Q1.3 (S)
- net at R8.3: now also U9.7 (IN-)
- net at U9.8 (IN+): now also R8.2
- net Shunt_IN: now reaches R8.4
- net Shunt_IN: now also D1.1 (K), Q1.3 (S)
Other:
- note added: "Como só temos um INA e o canal I2C a usar vai ser dedicado, qualquer configuração de A1 e A0 serve."
- note removed: "Confirmar mais tarde ligações a pinos A0/A1"
- note removed: "Ler datasheet para determinar valor do shunt"
- note removed: "Potencial filtragem. Tenho de confirmar se será necessário mas penso que não, o mais provável é deixar na PCB e logo decidir se meto componentes ou só dou bypass."
- moved on the sheet: R8

Commit message: Schematic update
- Add: SPI2 channel
- Add: INA I2C connections
- Component selection
Parts:
- removed J6, J7: Conn_01x03, symbol Connector_Generic:Conn_01x03
- C1, C17, C19, C2, C23, C25, C26, C28, C29, C3, C30, C32, C4, C5, C6, C7, C8: footprint (none) -> Capacitor_SMD:C_0603_1608Metric_Pad1.08x0.95mm_HandSolder; Mouser link (none) -> https://pt.mouser.com/ProductDetail/TAIYO-YUDEN/MAJCU168BB7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
- C22, C27: footprint (none) -> Capacitor_SMD:C_0603_1608Metric_Pad1.08x0.95mm_HandSolder
- R1, R12, R13, R14, R15, R16, R17, R18, R19, R20, R21, R5, R6: footprint (none) -> Resistor_SMD:R_0805_2012Metric_Pad1.20x1.40mm_HandSolder; Mouser link (none) -> https://pt.mouser.com/ProductDetail/YAGEO/RT0805FRE1010KL?q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
- R11: value R -> 150
- R4: Mouser link (none) -> https://pt.mouser.com/ProductDetail/YAGEO/RT0805FRE1010KL?q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
- R8: Mouser link (none) -> https://pt.mouser.com/ProductDetail/SEI-Stackpole/CSNL2512F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
- U1: Mouser link (none) -> https://eu.mouser.com/ProductDetail/Microchip-Technology/PI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
Connections:
- net Pyro_channel1 is gone; now on net Pyro1: Q2.2 (G), R14.2
- net Pyro_channel2 is gone; now on net Pyro2: Q3.2 (G), R13.2
- net Pyro_channel3 is gone; now on net Pyro3: Q4.2 (G), R15.2
- net Pyro_channel4 is gone; now on net Pyro4: Q5.2 (G), R16.2
- net ALT_CS: now also U1.8 (EBIWE/AN20/RPC3/PMWR/RC3)
- net GND: now also U6.2 (PS), U7.2 (D_SEL)
- net IMU_CS: now also U1.86 (EBID10/ETXD0/RPF1/PMD10/RF1)
- net MAG_CS: now also U1.85 (EBID11/ETXD1/RPF0/PMD11/RF0)
- net PWR_SDA: now also U1.67 (AETXEN/RPA15/SDA1/RA15); no longer U1.5 (EBID7/AN15/PMD7/RE7)
- net SERVO_1: now also U1.71 (EMDIO/AEMDIO/RPD0/RTCC/INT0/RD0)
- net SERVO_2: now also U1.70 (EMDC/AEMDC/RPD11/RD11)
- net SERVO_3: now also U1.69 (RPD10/SCK4/RD10)
- net SERVO_4: now also U1.68 (EBIA15/RPD9/PMCS2/PMA15/RD9)
- net Shunt_IN: now also R8.1; no longer R8.4
- net Shunt_OUT: now also R8.4; no longer R8.1
- net SPI2_CLK: now reaches U1.10 (AN14/C1IND/ECOL/RPG6/SCK2/RG6)
- net SPI2_MISO: now reaches U1.6 (EBIA6/AN22/RPC1/PMA6/RC1)
- net PWR_SCL: now reaches U1.66 (AETXCLK/RPA14/SCL1/RA14)
- net PWR_SCL: now also R19.1, U9.4 (SCL)
- net SPI2_MOSI: now reaches U1.7 (EBIA12/AN21/RPC2/PMA12/RC2)
- net Pyro3: now reaches U1.78 (EBID15/ETXCLK/RPD3/PMD15/RD3)
- net Pyro4: now reaches U1.79 (EBID12/ETXD2/RPD12/PMD12/RD12)
- net Pyro2: now reaches U1.81 (SQICS0/RPD4/RD4)
- net Pyro1: now reaches U1.82 (SQICS1/RPD5/RD5)
- removed net PWR_SDL: R19.1, U1.4 (EBID6/AN16/PMD6/RE6), U9.4 (SCL)
- net SPI_CLK renamed SPI1_CLK
- net SPI_MISO renamed SPI1_MISO
- net SPI_MOSI renamed SPI1_MOSI
Other:
- note added: "POWER IN"
- note added: "SPI1 - MAG & IMU SPI2 - ALT/TEMP (sensitive/recommended) SPI3 - GPS & LOGGING"
- note added: "SPI1 CLK"
- note added: "SPI1 MISO"
- note added: "SPI1 MOSI"
- note added: "SPI2 CLK"
- note added: "SPI2 MISO"
- note added: "SPI2 MOSI"
- note removed: "I2C"
- note removed: "SPI CLK"
- note removed: "SPI MISO"
- note removed: "SPI MOSI"
- note removed: "UART/DDC"
- note removed: "Vale a pena adicionar um conector para ligar uma bateria de backup? (3V3)"
- title: (none) -> Helios Flight Computer
- moved on the sheet: BT1, C15, C18, C19, C20, C21, C28, C29, C6, D1, F1, Q1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
