File: FC_Board/FC.kicad_pcb (KiCad board)
At the start: 2 copper layers, 98 parts, among them J1 Programmer_pins, J2 Pyro1, J3 Pyro2, J4 Pyro3, J5 Pyro4, J6 Conn_01x05, J7 USB_B_Micro, J8 MEM2090-00-145-00-A_REVA, M1 Motor_Servo, M2 Motor_Servo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

Commit message: Started PCB
Parts:
- C10, C11, C12, C13, C14, C15, C16, C9: moved to B.Cu
- moved BZ1 134.8 mm to (238.6, 99.4)
- moved C26 121.9 mm to (246.8, 111.6)
- moved C27 121.9 mm to (246.8, 114.1)
- moved C28 121.9 mm to (246.8, 116.6)
- moved C29 121.9 mm to (246.8, 119.1)
- moved C30 121.9 mm to (246.8, 121.6)
- moved C31 121.9 mm to (246.8, 124.1)
- moved C32 121.9 mm to (246.8, 126.6)
- moved C33 121.9 mm to (246.8, 129.2)
- moved R10 121.9 mm to (251.2, 116.6)
- moved R11 121.9 mm to (251.2, 119.1)
- moved R7 121.9 mm to (251.2, 111.6)
- moved R9 121.9 mm to (251.2, 114.1)
- moved D3 108.7 mm to (269.5, 87.0)
- moved J5 108.7 mm to (262.6, 21.7)
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Routing:
- added copper zone on B.Cu, net GND
- added copper zone on F.Cu, net GND

Commit message: First placement attempt
Parts:
- BT1: footprint Connector_AMASS:AMASS_XT60IPW-M_1x03_P7.20mm_Horizontal -> Connector_AMASS:AMASS_XT60-M_1x02_P7.20mm_Vertical
- C22, C27, C30, J8, R10, R13, R14, R15, R16, R18, R19, R20, R21, R22, R24, R4, R6, R9, U5: moved to B.Cu
- U2: footprint Package_TO_SOT_THT:TO-220-3_Horizontal_TabDown -> Package_TO_SOT_THT:TO-220-3_Vertical
- moved C24 157.1 mm to (214.6, 75.7), turned to -90 degrees
- moved J7 142.7 mm to (148.6, 111.3), turned to -90 degrees
- moved R22 142.6 mm to (156.5, 108.4)
- moved C19 138.8 mm to (199.8, 70.2), turned to -90 degrees
- moved U6 134.3 mm to (174.4, 121.0)
- moved C22 133.1 mm to (176.2, 99.8), turned to 180 degrees
- moved J8 132.1 mm to (216.4, 61.3)
- moved C23 131.4 mm to (177.8, 97.8)
- moved C17 125.4 mm to (171.5, 115.8), turned to 180 degrees
- moved U10 122.0 mm to (155.0, 111.4), turned to 90 degrees
- moved U11 121.5 mm to (151.7, 102.5), turned to 90 degrees
- moved J4 120.9 mm to (148.9, 78.8)
- moved J5 119.9 mm to (157.2, 78.8)
- moved M1 115.3 mm to (217.8, 80.9)
- moved Q2 114.9 mm to (150.5, 63.0), turned to 180 degrees
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Routing:
- net Battery_VDD: track 0.00 -> 50.2 mm
- net Shunt_OUT: track 0.00 -> 47.9 mm
- net Shunt_IN: track 0.00 -> 31.5 mm
- net Net-(BZ1--): track 0.00 -> 13.7 mm
- net Net-(Q1-D): track 0.00 -> 10.6 mm
- net Buzzer_pin: track 0.00 -> 8.32 mm
- net Net-(J4-Pin_2): track 0.00 -> 7.58 mm
- net V_BACKUP: track 0.00 -> 6.63 mm
- net Net-(J3-Pin_2): track 0.00 -> 5.67 mm
- net Net-(D1-A): track 0.00 -> 5.61 mm
- net Net-(J5-Pin_2): track 0.00 -> 4.97 mm
- net Net-(J2-Pin_2): track 0.00 -> 4.89 mm
- net Net-(D2-K): track 0.00 -> 3.13 mm
Other:
- board outline added: 80 x 65 mm

Commit message: Transitioning to 4 layers
Tried 2 layer routing to minimize cost. Too many tracks...
Parts:
- moved R12 4.05 mm to (210.8, 67.0), turned to 180 degrees
- moved R28 1.90 mm to (209.7, 63.5), turned to -90 degrees
- moved R27 1.74 mm to (212.5, 63.6), turned to -90 degrees
- moved C24 1.72 mm to (214.7, 77.4), turned to 90 degrees
- moved R25 1.64 mm to (219.8, 63.6), turned to -90 degrees
- moved R26 1.34 mm to (216.9, 63.6), turned to -90 degrees
- moved C32 1.18 mm to (215.1, 65.8)
Connections:
- U1 pad 10: SPI2_CLK -> ALT_CLK
- U1 pad 43: SPI3_CLK -> FLASH_CLK
- U1 pad 47: SPI3_MISO -> FLASH_SO
- U1 pad 48: SPI3_MOSI -> FLASH_SI
- U1 pad 6: SPI2_MISO -> ALT_SDO
- U1 pad 7: SPI2_MOSI -> ALT_SDI
- U1 pad 72: SPI1_MOSI -> IMU_SDI
- U1 pad 73: SPI1_MISO -> IMU_SDO
- U1 pad 76: SPI1_CLK -> IMU_CLK
- U1 pad 89: SPI4_CLK -> SD_CLK
- U1 pad 90: SPI4_SIO3 -> SD_D3
- U1 pad 95: SPI4_SIO2 -> SD_D2
- U1 pad 96: SPI4_SIO1 -> SD_D1
- U1 pad 97: SPI4_SIO0 -> SD_D0
- U5 pad 1: MAG_CLK -> IMU_CLK
- U5 pad 11: MAG_SDI -> IMU_SDI
- U5 pad 9: MAG_SDO -> IMU_SDO
- U7 pad 19: GPS_CLK -> FLASH_CLK
- U7 pad 20: GPS_TXD -> FLASH_SO
- U7 pad 21: GPS_RXD -> FLASH_SI
Routing:
- net Battery_VDD: track 50.2 -> 0.00 mm
- net Shunt_OUT: track 47.9 -> 0.00 mm
- net Shunt_IN: track 31.5 -> 0.00 mm
- net Net-(BZ1--): track 13.7 -> 0.00 mm
- net Net-(Q1-D): track 10.6 -> 0.00 mm
- net Buzzer_pin: track 8.32 -> 0.00 mm
- net Net-(J4-Pin_2): track 7.58 -> 0.00 mm
- net V_BACKUP: track 6.63 -> 0.00 mm
- net Net-(J3-Pin_2): track 5.67 -> 0.00 mm
- net Net-(D1-A): track 5.61 -> 0.00 mm
- net Net-(J5-Pin_2): track 4.97 -> 0.00 mm
- net Net-(J2-Pin_2): track 4.89 -> 0.00 mm
- net Net-(D2-K): track 3.13 -> 0.00 mm
- added copper zone on In1.Cu, net GND
- added copper zone on In2.Cu, net GND
Other:
- copper layers 2 -> 4

Commit message: Routing done except for gnd vias
Parts:
- removed C2: 0.1uF, Capacitor_SMD:C_0603_1608Metric_Pad1.08x0.95mm_HandSolder
- C33: moved to B.Cu
- R13, R14, R15, R16: moved to F.Cu
- moved C33 6.08 mm to (153.9, 100.5), turned to -90 degrees
- moved C29 2.89 mm to (206.6, 110.5), turned to -90 degrees
- moved R5 1.08 mm to (182.4, 91.5)
- moved R11 0.99 mm to (160.8, 89.6)
- moved Q4 0.80 mm to (155.3, 84.2)
- moved R16 0.65 mm to (163.4, 87.2)
- moved R10 0.55 mm to (153.7, 93.2)
- moved Q5 0.54 mm to (160.7, 84.2)
- moved J5 0.38 mm to (157.5, 78.8)
- moved AE1 0.21 mm to (148.1, 94.3)
- moved J7 0.16 mm to (148.7, 111.2)
- moved C18 0.10 mm to (200.1, 65.0)
- moved J4 0.07 mm to (149.0, 78.8)
- turned R15 to 0 degrees
Routing:
- net 3V3: track 0.00 -> 120.4 mm, vias 0 -> 31
- net SD_D3: track 0.00 -> 78.2 mm, vias 0 -> 4
- net SD_D2: track 0.00 -> 65.7 mm, vias 0 -> 5
- net SD_IN#: track 0.00 -> 65.3 mm, vias 0 -> 3
- net SD_CMD: track 0.00 -> 64.7 mm, vias 0 -> 4
- net 5V: track 0.00 -> 63.8 mm
- net SD_D0: track 0.00 -> 62.1 mm, vias 0 -> 3
- net IMU_CLK: track 0.00 -> 61.7 mm, vias 0 -> 6
- net Pyro1: track 0.00 -> 60.0 mm, vias 0 -> 2
- net SD_CLK: track 0.00 -> 60.0 mm, vias 0 -> 5
- net FLASH_CLK: track 0.00 -> 59.9 mm, vias 0 -> 5
- net SD_D1: track 0.00 -> 59.3 mm, vias 0 -> 5
- net IMU_SDO: track 0.00 -> 56.6 mm, vias 0 -> 4
- net Battery_VDD: track 0.00 -> 55.9 mm
- net FLASH_SI: track 0.00 -> 55.3 mm, vias 0 -> 3
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- added copper zone on In1.Cu, net 3V3
- added copper zone on In2.Cu, net 3V3
- removed copper zone on In1.Cu, net GND
- removed copper zone on In2.Cu, net GND

Commit message: Helios_v1.0 DONE
Parts:
- added G***: LOGO, Graphics_helios:Helios_symbol, F.Cu at (210.0, 101.7)
Routing:
- net 3V3: track 120.4 -> 130.2 mm
- net Net-(C17-Pad1): track 2.34 -> 4.75 mm
- net GND: track 27.7 -> 29.0 mm, vias 15 -> 201
Other:
- board text added: "RC"
